Commit message: QS Profile adjusted, TODO: Add more waypoints

File: dbw_gazebo_mkz/urdf/mkz.urdf.xacro (robot description, xacro)
@@ -1,183 +1,16 @@
 <?xml version="1.0"?>
-<!-- created with Phobos 0.7 -->
-  <robot name="dbw_mkz" xmlns:xacro="http://www.ros.org/wiki/xacro">
-    <xacro:arg name="dae_file" default="$(find dataspeed_dbw_gazebo)/urdf/mkz/meshes/body.dae"/>
-    <link name="base_footprint">
-    </link>
-    <link name="base_link">
-      <inertial>
-        <origin xyz="1.4225 0 0.25" rpy="0 0 0"/>
-        <mass value="1500.0"/>
-        <inertia ixx="1000.0" ixy="0" ixz="0" iyy="1000.0" iyz="0" izz="1000.0"/>
-      </inertial>
-      <visual name="chassis">
-        <origin xyz="1.39 0 -0.371498" rpy="0 0 1.570796"/>
-        <geometry>
-          <mesh filename="file://$(arg dae_file)" scale="1 0.97 1"/>
-        </geometry>
-        <material name="black.001"/>
-      </visual>
-      <collision name="chassis_collision">
-        <origin xyz="1.4768 -0.019748 0.332734" rpy="1.570796 0 -3.141593"/>
-        <geometry>
-          <mesh filename="file://$(find dataspeed_dbw_gazebo)/urdf/mkz/meshes/body_collision.stl" scale="0.001 0.001 0.001"/>
-        </geometry>
-      </collision>
-    </link>
-    <link name="steer_fl">
-      <inertial>
-        <origin xyz="0 0 0" rpy="0 0 0"/>
-        <mass value="1.0"/>
-        <inertia ixx="0.037227" ixy="0" ixz="0" iyy="0.04" iyz="0" izz="0.06"/>
-      </inertial>
-    </link>
-    <link name="steer_fr">
-      <inertial>
-        <origin xyz="0 0 0" rpy="0 0 0"/>
-        <mass value="1.0"/>
-        <inertia ixx="0.037227" ixy="0" ixz="0" iyy="0.04" iyz="0" izz="0.06"/>
-      </inertial>
-    </link>
-    <link name="wheel_fl">
-      <inertial>
-        <origin xyz="0 0 0" rpy="0 -3.141593 0"/>
-        <mass value="10.0"/>
-        <inertia ixx="0.305583" ixy="0" ixz="0" iyy="0.305583" iyz="0" izz="0.5445"/>
-      </inertial>
-      <visual name="wheel_fl_visual">
-        <origin xyz="-0.0026 0 0.017813" rpy="-1.570796 1.570796 0"/>
-        <geometry>
-          <mesh filename="file://$(find dataspeed_dbw_gazebo)/urdf/mkz/meshes/wheel.dae" scale="0.01 0.01 0.01"/>
-        </geometry>
-        <material name="carpaint_002"/>
-      </visual>
-      <collision name="wheel_fl_collision">
-        <origin xyz="0 0 0" rpy="0 -3.141593 0"/>
-        <geometry>
-          <cylinder radius="0.33" length="0.2"/>
-        </geometry>
-      </collision>
-    </link>
-    <link name="wheel_fr">
-      <inertial>
-        <origin xyz="0 0 0" rpy="0 3.141593 0"/>
-        <mass value="10.0"/>
-        <inertia ixx="0.305583" ixy="0" ixz="0" iyy="0.305583" iyz="0" izz="0.5445"/>
-      </inertial>
-      <visual name="wheel_fr_visual">
-        <origin xyz="-0.0026 0 -0.0217" rpy="-1.570796 -1.570796 0"/>
-        <geometry>
-          <mesh filename="file://$(find dataspeed_dbw_gazebo)/urdf/mkz/meshes/wheel.dae" scale="0.01 0.01 0.01"/>
-        </geometry>
-        <material name="carpaint_002.001"/>
-      </visual>
-      <collision name="wheel_fr_collision">
-        <origin xyz="0 0 -0.0035" rpy="0 3.141593 0"/>
-        <geometry>
-          <cylinder radius="0.33" length="0.2"/>
-        </geometry>
-      </collision>
-    </link>
-    <link name="wheel_rl">
-      <inertial>
-        <origin xyz="0 0 -0.021117" rpy="0 3.141593 0"/>
-        <mass value="10.0"/>
-        <inertia ixx="0.305583" ixy="0" ixz="0" iyy="0.305583" iyz="0" izz="0.5445"/>
-      </inertial>
-      <visual name="wheel_rl_visual">
-        <origin xyz="0.0026 0 -0.00412" rpy="-1.570796 1.570796 0"/>
-        <geometry>
-          <mesh filename="file://$(find dataspeed_dbw_gazebo)/urdf/mkz/meshes/wheel.dae" scale="0.01 0.01 0.01"/>
-        </geometry>
-        <material name="carpaint_002.003"/>
-      </visual>
-      <collision name="wheel_rl_collision">
-        <origin xyz="0 0 -0.021118" rpy="0 3.141593 0"/>
-        <geometry>
-          <cylinder radius="0.33" length="0.2"/>
-        </geometry>
-      </collision>
-    </link>
-    <link name="wheel_rr">
-      <inertial>
-        <origin xyz="0 0 0.0205" rpy="0 3.141593 0"/>
-        <mass value="10.0"/>
-        <inertia ixx="0.305583" ixy="0" ixz="0" iyy="0.305583" iyz="0" izz="0.5445"/>
-      </inertial>
-      <visual name="wheel_rr_visual">
-        <origin xyz="0.0026 0 0.00331" rpy="-1.570796 -1.570796 0"/>
-        <geometry>
-          <mesh filename="file://$(find dataspeed_dbw_gazebo)/urdf/mkz/meshes/wheel.dae" scale="0.01 0.01 0.01"/>
-        </geometry>
-        <material name="carpaint_002.002"/>
-      </visual>
-      <collision name="wheel_rr_collision">
-        <origin xyz="0 0 0.0205" rpy="0 3.141593 0"/>
-        <geometry>
-          <cylinder radius="0.33" length="0.2"/>
-        </geometry>
-      </collision>
-    </link>
-    <joint name="base_link_joint" type="fixed">
-      <origin xyz="0 0 0.33" rpy="0 0 0"/>
-      <parent link="base_footprint"/>
-      <child link="base_link"/>
-    </joint>
-    <joint name="steer_fl_joint" type="revolute">
-      <origin xyz="2.85 0.79712 0" rpy="0 0 0"/>
-      <parent link="base_link"/>
-      <child link="steer_fl"/>
-      <axis xyz="0 0 1.0"/>
-      <limit lower="-0.6" upper="0.6" effort="-1.0" velocity="-1.0"/>
-    </joint>
-    <joint name="steer_fr_joint" type="revolute">
-      <origin xyz="2.85 -0.79712 0.0" rpy="0 0 0"/>
-      <parent link="base_link"/>
-      <child link="steer_fr"/>
-      <axis xyz="0 0 1.0"/>
-      <limit lower="-0.6" upper="0.6" effort="-1.0" velocity="-1.0"/>
-    </joint>
-    <joint name="wheel_fl_joint" type="continuous">
-      <origin xyz="0 0 0" rpy="1.570796 0 -3.141593"/>
-      <parent link="steer_fl"/>
-      <child link="wheel_fl"/>
-      <axis xyz="0 0 1.0"/>
-      <limit effort="-1.0" velocity="-1.0"/>
-    </joint>
-    <joint name="wheel_fr_joint" type="continuous">
-      <origin xyz="0 0 0" rpy="1.570796 0 -3.141593"/>
-      <parent link="steer_fr"/>
-      <child link="wheel_fr"/>
-      <axis xyz="0 0 1.0"/>
-      <limit effort="-1.0" velocity="-1.0"/>
-    </joint>
-    <joint name="wheel_rl_joint" type="continuous">
-      <origin xyz="0 0.7874 0" rpy="1.570796 0 -3.141593"/>
-      <parent link="base_link"/>
-      <child link="wheel_rl"/>
-      <axis xyz="0 0 1.0"/>
-      <limit effort="-1.0" velocity="-1.0"/>
-    </joint>
-    <joint name="wheel_rr_joint" type="continuous">
-      <origin xyz="0 -0.7874 0" rpy="1.570796 0 -3.141593"/>
-      <parent link="base_link"/>
-      <child link="wheel_rr"/>
-      <axis xyz="0 0 1.0"/>
-      <limit effort="-1.0" velocity="-1.0"/>
-    </joint>
-    <material name="black.001">
-      <color rgba="0 0 0 1.0"/>
-    </material>
-    <material name="carpaint_002">
-      <color rgba="0.941177 0.941177 0.941177 1.0"/>
-    </material>
-    <material name="carpaint_002.001">
-      <color rgba="0.941177 0.941177 0.941177 1.0"/>
-    </material>
-    <material name="carpaint_002.002">
-      <color rgba="0.941177 0.941177 0.941177 1.0"/>
-    </material>
-    <material name="carpaint_002.003">
-      <color rgba="0.941177 0.941177 0.941177 1.0"/>
-    </material>
-  </robot>
+<robot name="mkz" xmlns:xacro="http://www.ros.org/wiki/xacro" >
+  <!-- Necessary includes -->
+  <xacro:include filename="$(arg structure_urdf)" />
+  <xacro:include filename="$(find dataspeed_dbw_gazebo)/urdf/vehicle_gazebo.urdf.xacro" />
+  <!-- Bolt-on sensors go here -->
+  <xacro:include filename="$(find custom_dbw_sim_examples)/urdf/vehicle_sensors.urdf.xacro" />
+  <xacro:dataspeed_dbw_gazebo_camera name="front_camera" parent="base_footprint" >
+    <origin xyz="2.1 0 1.4" rpy="0 0.55 0" />
+  </xacro:dataspeed_dbw_gazebo_camera>
+  <xacro:dataspeed_dbw_gazebo_gps name="perfect_gps" parent="base_footprint" x="0.6" y="0" z="1.45" rate="50.0" ref_lat="45.0" ref_lon="-81.0" />
+  <xacro:include filename="$(find velodyne_description)/urdf/VLP-16.urdf.xacro"/>
+  <xacro:VLP-16 parent="base_footprint" name="velodyne" topic="velodyne_points" hz="10" samples="440">
+    <origin xyz="1.1 0 1.49" rpy="0 0 0" />
+  </xacro:VLP-16>
+</robot>
