Commit message: changes to RVIZ plugin and Waypoint Plotter

File: src/dbw_gazebo_mkz/urdf/mkz.urdf.xacro (robot description, xacro)
@@ -10,7 +10,4 @@
   </xacro:dataspeed_dbw_gazebo_camera>
   <xacro:dataspeed_dbw_gazebo_gps name="perfect_gps" parent="base_footprint" x="0.6" y="0" z="1.45" rate="50.0" ref_lat="45.0" ref_lon="-81.0" />
-  <xacro:include filename="$(find velodyne_description)/urdf/VLP-16.urdf.xacro"/>
-  <xacro:VLP-16 parent="base_footprint" name="velodyne" topic="velodyne_points" hz="10" samples="440">
-    <origin xyz="1.1 0 1.49" rpy="0 0 0" />
-  </xacro:VLP-16>
+  <xacro:imu_link name="imu_link" parent="base_footprint" x="1.6" y="0" z="1.45" rpy="0 0 0"/>
 </robot>

File: src/dbw_gazebo_mkz/urdf/vehicle_sensors.urdf.xacro (robot description, xacro)
@@ -106,3 +106,52 @@
     </gazebo>
   </xacro:macro>
+  <xacro:macro name="imu_link" params="name rpy parent x y z " >
+    <link name="${name}" >
+      <visual>
+        <origin xyz="0 0 0" rpy="0 0 0" />
+        <geometry>
+          <cylinder radius="0.1" length="0.05" />
+        </geometry>
+        <material name="white" >
+          <color rgba="1 1 1 1" />
+        </material>
+      </visual>
+      <collision>
+        <origin xyz="0 0 0" rpy="0 0 0" />
+        <geometry>
+          <cylinder radius="0.1" length="0.05" />
+        </geometry>
+      </collision>
+      <inertial>
+        <origin xyz="0 0 0" rpy="0 0 0"/>
+        <mass value="1.0"/>
+        <inertia ixx="0.037227" ixy="0" ixz="0" iyy="0.037227" iyz="0" izz="0.063878"/>
+      </inertial>
+    </link>
+    <joint name="${name}" type="fixed" >
+      <origin xyz="${x} ${y} ${z}" rpy="0 0 0" />
+      <parent link="${parent}" />
+      <child link="${name}" />
+    </joint>
+    <gazebo reference="imu_link">
+    <gravity>true</gravity>
+    <sensor name="imu_sensor" type="imu">
+      <always_on>true</always_on>
+      <update_rate>100</update_rate>
+      <visualize>true</visualize>
+      <topic>__default_topic__</topic>
+      <plugin filename="libgazebo_ros_imu_sensor.so" name="imu_plugin">
+        <topicName>imu</topicName>
+        <bodyName>imu_link</bodyName>
+        <updateRateHZ>10.0</updateRateHZ>
+        <gaussianNoise>0.0</gaussianNoise>
+        <xyzOffset>0 0 0</xyzOffset>
+        <rpyOffset>0 0 0</rpyOffset>
+        <frameName>imu_link</frameName>
+        <initialOrientationAsReference>false</initialOrientationAsReference>
+      </plugin>
+      <pose>0 0 0 0 0 0</pose>
+    </sensor>
+  </gazebo>
+ </xacro:macro>
 </robot>
